Commit message: Model gripper (optional with arg)
This commit also modifies the ultrasonic sensor definition to
allow its proper placement when combining it with the gripper.

File: mark_description/urdf/mark.urdf.xacro (robot description, xacro)
@@ -3,4 +3,5 @@
   <!-- Parameters -->
   <xacro:arg name="ultrasonic_sensor_enabled" default="true" />
+  <xacro:arg name="gripper_enabled" default="true" />
   <!-- Includes -->
   <xacro:include filename="$(find mark_description)/urdf/inertial.urdf.xacro" />
@@ -10,4 +11,5 @@
   <xacro:include filename="$(find mark_description)/urdf/camera.urdf.xacro" />
   <xacro:include filename="$(find mark_description)/urdf/ultrasonic.urdf.xacro" />
+  <xacro:include filename="$(find mark_description)/urdf/gripper.urdf.xacro" />
   <!-- Base/chassis -->
   <xacro:mark_base></xacro:mark_base>
@@ -25,10 +27,22 @@
   <!-- Ultrasonic sensor (if requied) -->
   <xacro:if value="$(arg ultrasonic_sensor_enabled)">
-    <xacro:mark_ultrasonic_sensor>
-      <origin xyz="0.083 0.0 -0.006" rpy="0 0 0" />
-    </xacro:mark_ultrasonic_sensor>
+    <!-- If the gripper is also enabled then place the ultrasonic sensor on the base of the gripper -->
+    <xacro:if value="$(arg gripper_enabled)">
+      <xacro:mark_ultrasonic_sensor parent="gripper_base_link">
+        <origin xyz="0.069 0.0 0.016" rpy="0 0 0" />
+      </xacro:mark_ultrasonic_sensor>
+    </xacro:if>
+    <!-- If the gripper is not enabled then place the ultrasonic sensor on the base of the robot -->
+    <xacro:unless value="$(arg gripper_enabled)">
+      <xacro:mark_ultrasonic_sensor parent="base_link">
+        <origin xyz="0.084 0.0 -0.003" rpy="0 0 0" />
+      </xacro:mark_ultrasonic_sensor>
+    </xacro:unless>
   </xacro:if>
-  <!-- TODO:
-       - Gripper (controller by arg)
-  -->
+  <!-- Gripper (if required) -->
+  <xacro:if value="$(arg gripper_enabled)">
+    <xacro:mark_gripper>
+      <origin xyz="0.03 0.0 -0.018" rpy="0 0 0" />
+    </xacro:mark_gripper>
+  </xacro:if>
 </robot>

File: mark_description/urdf/ultrasonic.urdf.xacro (robot description, xacro)
@@ -1,6 +1,6 @@
-<robot xmlns:xacro="http://ros.org/wiki/xacro" name="mark_wheel">
+<robot xmlns:xacro="http://ros.org/wiki/xacro" name="mark_ultrasonic">
   <xacro:property name="ultrasonic_sensor_base_geom">
     <geometry>
-      <box size="0.001 0.047 0.023" />
+      <box size="0.001 0.047 0.03" />
     </geometry>
   </xacro:property>
@@ -18,9 +18,9 @@
   <xacro:property name="ultrasonic_sensor_right_joint_pose">
     <!-- Rotate 90 degrees (in radians) -->
-    <origin xyz="0.008 0.012 0" rpy="0 1.560795 0" />
+    <origin xyz="0.0076 0.012 -0.005" rpy="0 1.560795 0" />
   </xacro:property>
   <xacro:property name="ultrasonic_sensor_left_joint_pose">
     <!-- Rotate 90 degrees (in radians) -->
-    <origin xyz="0.008 -0.012 0" rpy="0 1.560795 0" />
+    <origin xyz="0.0076 -0.012 -0.005" rpy="0 1.560795 0" />
   </xacro:property>
   <xacro:property name="ultrasonic_sensor_inertia">
@@ -49,5 +49,5 @@
   </xacro:macro>
   <!-- Full ultrasonic sensor macro-->
-  <xacro:macro name="mark_ultrasonic_sensor" params="*ultrasonic_sensor_base_joint_pose">
+  <xacro:macro name="mark_ultrasonic_sensor" params="parent *ultrasonic_sensor_base_joint_pose">
     <link name="ultrasonic_sensor_base_link">
       <visual>
@@ -60,6 +60,6 @@
       <xacro:insert_block name="ultrasonic_sensor_base_inertia" />
     </link>
-    <joint name="ultrasonic_sensor_base_to_robot_base_link" type="fixed">
-      <parent link="base_link" />
+    <joint name="ultrasonic_sensor_base_to_parent_link" type="fixed">
+      <parent link="${parent}" />
       <child link="ultrasonic_sensor_base_link" />
       <xacro:insert_block name="ultrasonic_sensor_base_joint_pose" />
