Commit message: Match chassis/wheel dimensions to the real ones
I manually measured the robot to make sure the model matches
the real dimensions as close as possible.

File: mark_description/urdf/base.urdf.xacro (robot description, xacro)
@@ -1,20 +1,24 @@
 <robot xmlns:xacro="http://ros.org/wiki/xacro" name="mark_base">
-  <!-- MARK dimensions: 200 * 185 * 92 mm  (D * W * H)-->
-  <xacro:property name="base_size" value="0.2 0.185 0.092" />
+  <!-- MARK dimensions:
+       - Length/Depth: 16.6cm (0.166m)
+       - Width: 12.5cm (0.125m)
+       - Height: 3.6cm (0.036m)
+  -->
+  <xacro:property name="base_size" value="0.166 0.125 0.036" />
   <!-- MARK weighs around 620g -->
-  <xacro:property name="base_weight" value="0.64" />
+  <xacro:property name="base_weight" value="0.62" />
   <!-- Inertia calculated using formulas here:
        https://en.wikipedia.org/wiki/List_of_moments_of_inertia#List_of_3D_inertia_tensors  -->
   <xacro:property name="base_inertia">
-    <inertia ixx="0.0025" ixy="0.0" ixz="0.0" iyy="0.0038" iyz="0.0" izz="0.0022"/>
+    <inertia ixx="0.0015" ixy="0.0" ixz="0.0" iyy="0.0022" iyz="0.0" izz="0.00087"/>
   </xacro:property>
   <!-- Caster (i.e. back support) -->
-  <xacro:property name="caster_origin" value="-0.038 0 -0.02" />
-  <xacro:property name="caster_radius" value="0.025" />
+  <xacro:property name="caster_origin" value="-0.037 0 -0.01" />
+  <xacro:property name="caster_radius" value="0.010" />
   <xacro:property name="caster_weight" value="0.5" />
   <xacro:property name="caster_inertia">
-    <inertia ixx="0.000125" ixy="0.0" ixz="0.0" iyy="0.000125" iyz="0.0" izz="0.000125"/>
+    <inertia ixx="0.00002" ixy="0.0" ixz="0.0" iyy="0.00002" iyz="0.0" izz="0.00002"/>
   </xacro:property>
-  <material name="black">
+  <material name="grey">
     <color rgba="0.45 0.45 0.45 1.0"/>
   </material>
@@ -27,5 +31,5 @@
           <box size="${base_size}" />
         </geometry>
-        <material name="black" />
+        <material name="grey" />
       </visual>
       <collision>
@@ -56,5 +60,5 @@
           <sphere radius="${caster_radius}" />
         </geometry>
-        <material name="black" />
+        <material name="grey" />
       </visual>
       <collision>

File: mark_description/urdf/mark.urdf.xacro (robot description, xacro)
@@ -8,8 +8,8 @@
   <!-- Wheels -->
   <xacro:mark_wheel wheel_prefix="right">
-    <origin xyz="0.03 0.1 -0.03" rpy="0 0 0" />
+    <origin xyz="0.045 0.075 -0.005" rpy="0 0 0" />
   </xacro:mark_wheel>
   <xacro:mark_wheel wheel_prefix="left">
-    <origin xyz="0.03 -0.1 -0.03" rpy="0 0 0" />
+    <origin xyz="0.045 -0.075 -0.005" rpy="0 0 0" />
   </xacro:mark_wheel>
   <!-- TODO:

File: mark_description/urdf/wheel.urdf.xacro (robot description, xacro)
@@ -1,33 +1,33 @@
 <robot xmlns:xacro="http://ros.org/wiki/xacro" name="mark_wheel">
-  <!-- We use `*` for the joint_pose to specify it's a block property
+  <!-- We use `*` for the joint_pose to specify it's a `block` property
        See: http://wiki.ros.org/xacro#Macros
   -->
   <xacro:macro name="mark_wheel" params="wheel_prefix *joint_pose">
-    <link name="${wheel_prefix}_wheel">
-    <visual>
-      <origin xyz="0 0 0" rpy="0 0 0" />
-      <geometry>
-        <mesh filename="package://mark_description/meshes/wheel.dae" />
-      </geometry>
-    </visual>
-    <collision>
-      <!-- The cylinder for the collision needs to be rotated 90 degrees (in radians) -->
-      <origin xyz="0 0 0" rpy="1.560795 0 0" />
-      <geometry>
-          <cylinder length="0.1" radius="0.2" />
-      </geometry>
-    </collision>
-    <inertial>
-      <mass value="0.5"/>
-      <inertia ixx="0.01" ixy="0.0" ixz="0.0" iyy="0.005" iyz="0.0" izz="0.005"/>
-    </inertial>
+    <link name="${wheel_prefix}_wheel_link">
+      <visual>
+        <origin xyz="0 0 0" rpy="0 0 0" />
+        <geometry>
+          <mesh filename="package://mark_description/meshes/wheel.dae" />
+        </geometry>
+      </visual>
+      <collision>
+        <!-- The cylinder for the collision needs to be rotated 90 degrees (in radians) -->
+        <origin xyz="0 0 0" rpy="1.560795 0 0" />
+        <geometry>
+          <cylinder length="0.062" radius="0.031" />
+        </geometry>
+      </collision>
+      <inertial>
+        <mass value="0.5" />
+        <inertia ixx="0.00028" ixy="0.0" ixz="0.0" iyy="0.00028" iyz="0.0" izz="0.00024" />
+      </inertial>
     </link>
     <joint name="joint_${wheel_prefix}_wheel" type="continuous">
-      <parent link="chassis_link"/>
-      <child link="${wheel_prefix}_wheel"/>
+      <parent link="base_link"/>
+      <child link="${wheel_prefix}_wheel_link"/>
       <xacro:insert_block name="joint_pose"/>
       <!-- Rotation on the y-axis -->
       <axis xyz="0 1 0" />
-  </joint>
+    </joint>
   </xacro:macro>
 </robot>

Commit message: Fix caster pose
Visual/collision should be in the origin and the joint should be
moved to where we want the link to be

File: mark_description/urdf/base.urdf.xacro (robot description, xacro)
@@ -14,5 +14,5 @@
   </xacro:property>
   <!-- Caster (i.e. back support) -->
-  <xacro:property name="caster_origin" value="-0.037 0 -0.01" />
+  <xacro:property name="caster_origin" value="-0.073 0 -0.02" />
   <xacro:property name="caster_radius" value="0.010" />
   <xacro:property name="caster_weight" value="0.5" />
@@ -56,5 +56,5 @@
     <link name="caster_link">
       <visual>
-        <origin xyz="${caster_origin}" rpy="0 0 0" />
+        <origin xyz="0 0 0" rpy="0 0 0" />
         <geometry>
           <sphere radius="${caster_radius}" />
@@ -63,5 +63,5 @@
       </visual>
       <collision>
-        <origin xyz="${caster_origin}" rpy="0 0 0" />
+        <origin xyz="0 0 0" rpy="0 0 0" />
         <geometry>
           <sphere radius="${caster_radius}" />

Commit message: Model camera w/ pan/tilt movement

File: mark_description/urdf/base.urdf.xacro (robot description, xacro)
@@ -20,7 +20,4 @@
     <inertia ixx="0.00002" ixy="0.0" ixz="0.0" iyy="0.00002" iyz="0.0" izz="0.00002"/>
   </xacro:property>
-  <material name="grey">
-    <color rgba="0.45 0.45 0.45 1.0"/>
-  </material>
   <xacro:macro name="mark_base">
     <!-- Base -->

File: mark_description/urdf/mark.urdf.xacro (robot description, xacro)
@@ -2,6 +2,9 @@
 <robot name="mark" xmlns:xacro="http://ros.org/wiki/xacro">
   <!-- Includes -->
+  <xacro:include filename="$(find mark_description)/urdf/inertial.urdf.xacro" />
+  <xacro:include filename="$(find mark_description)/urdf/materials.urdf.xacro" />
   <xacro:include filename="$(find mark_description)/urdf/base.urdf.xacro" />
   <xacro:include filename="$(find mark_description)/urdf/wheel.urdf.xacro" />
+  <xacro:include filename="$(find mark_description)/urdf/camera.urdf.xacro" />
   <!-- Base/chassis -->
   <xacro:mark_base></xacro:mark_base>
@@ -13,8 +16,11 @@
     <origin xyz="0.045 -0.075 -0.005" rpy="0 0 0" />
   </xacro:mark_wheel>
+  <!-- Camera -->
+  <xacro:mark_camera>
+    <origin xyz="0.06 0.0 0.023" rpy="0 0 0" />
+  </xacro:mark_camera>
   <!-- TODO:
-       1. Camera
-       2. Ultrasonic sensor (controlled by arg)
-       3. Gripper (controller by arg)
+       - Ultrasonic sensor (controlled by arg)
+       - Gripper (controller by arg)
   -->
 </robot>

File: mark_description/urdf/wheel.urdf.xacro (robot description, xacro)
@@ -24,7 +24,7 @@
     </link>
     <joint name="joint_${wheel_prefix}_wheel" type="continuous">
-      <parent link="base_link"/>
-      <child link="${wheel_prefix}_wheel_link"/>
-      <xacro:insert_block name="joint_pose"/>
+      <parent link="base_link" />
+      <child link="${wheel_prefix}_wheel_link" />
+      <xacro:insert_block name="joint_pose" />
       <!-- Rotation on the y-axis -->
       <axis xyz="0 1 0" />

Commit message: Standardize use of inertial macros + other cleanup

File: mark_description/urdf/base.urdf.xacro (robot description, xacro)
@@ -1,22 +1,23 @@
 <robot xmlns:xacro="http://ros.org/wiki/xacro" name="mark_base">
-  <!-- MARK dimensions:
-       - Length/Depth: 16.6cm (0.166m)
-       - Width: 12.5cm (0.125m)
-       - Height: 3.6cm (0.036m)
-  -->
-  <xacro:property name="base_size" value="0.166 0.125 0.036" />
-  <!-- MARK weighs around 620g -->
-  <xacro:property name="base_weight" value="0.62" />
-  <!-- Inertia calculated using formulas here:
-       https://en.wikipedia.org/wiki/List_of_moments_of_inertia#List_of_3D_inertia_tensors  -->
+  <xacro:property name="base_geom">
+    <geometry>
+      <box size="0.166 0.125 0.036" />
+    </geometry>
+  </xacro:property>
   <xacro:property name="base_inertia">
-    <inertia ixx="0.0015" ixy="0.0" ixz="0.0" iyy="0.0022" iyz="0.0" izz="0.00087"/>
+    <inertial>
+      <mass value="0.62" />
+      <xacro:box_inertia m="0.62" d="0.166" w="0.125" h="0.036" />
+    </inertial>
   </xacro:property>
-  <!-- Caster (i.e. back support) -->
   <xacro:property name="caster_origin" value="-0.073 0 -0.02" />
-  <xacro:property name="caster_radius" value="0.010" />
-  <xacro:property name="caster_weight" value="0.5" />
-  <xacro:property name="caster_inertia">
-    <inertia ixx="0.00002" ixy="0.0" ixz="0.0" iyy="0.00002" iyz="0.0" izz="0.00002"/>
+  <xacro:property name="caster_geom">
+    <sphere radius="0.010" />
+  </xacro:property>
+  <xacro:property name="base_inertia">
+    <inertial>
+      <mass value="0.5" />
+      <xacro:sphere_inertia m="0.5" r="0.010" />
+    </inertial>
   </xacro:property>
   <xacro:macro name="mark_base">
@@ -24,15 +25,9 @@
     <link name="base_link">
       <visual>
-        <origin xyz="0 0 0" rpy="0 0 0" />
-        <geometry>
-          <box size="${base_size}" />
-        </geometry>
+        <xacro:insert_block name="base_geom" />
         <material name="grey" />
       </visual>
       <collision>
-        <origin xyz="0 0 0" rpy="0 0 0" />
-        <geometry>
-          <box size="${base_size}"/>
-        </geometry>
+        <xacro:insert_block name="base_geom" />
       </collision>
     </link>
@@ -40,11 +35,7 @@
          Has to be defined separately because root links can't have intertial information directly -->
     <link name="inertial_link">
-      <inertial>
-        <mass value="${base_weight}"/>
-        <xacro:insert_block name="base_inertia" />
-      </inertial>
+      <xacro:insert_block name="base_inertia" />
     </link>
     <joint name="inertial_joint" type="fixed">
-      <origin xyz="0 0 0" rpy="0 0 0" />
       <parent link="base_link" />
       <child link="inertial_link" />
@@ -53,20 +44,11 @@
     <link name="caster_link">
       <visual>
-        <origin xyz="0 0 0" rpy="0 0 0" />
-        <geometry>
-          <sphere radius="${caster_radius}" />
-        </geometry>
+        <xacro:insert_block name="caster_geom" />
         <material name="grey" />
       </visual>
       <collision>
-        <origin xyz="0 0 0" rpy="0 0 0" />
-        <geometry>
-          <sphere radius="${caster_radius}" />
-        </geometry>
+        <xacro:insert_block name="caster_geom" />
       </collision>
-      <inertial>
-        <mass value="${caster_weight}"/>
-        <xacro:insert_block name="caster_inertia" />
-      </inertial>
+      <xacro:insert_block name="caster_inertial" />
     </link>
     <joint name="caster_to_base_joint" type="fixed">

File: mark_description/urdf/wheel.urdf.xacro (robot description, xacro)
@@ -6,5 +6,4 @@
     <link name="${wheel_prefix}_wheel_link">
       <visual>
-        <origin xyz="0 0 0" rpy="0 0 0" />
         <geometry>
           <mesh filename="package://mark_description/meshes/wheel.dae" />
@@ -20,5 +19,5 @@
       <inertial>
         <mass value="0.5" />
-        <inertia ixx="0.00028" ixy="0.0" ixz="0.0" iyy="0.00028" iyz="0.0" izz="0.00024" />
+        <xacro:cylinder_inertia m="0.5" r="0.031" h="0.062" />
       </inertial>
     </link>
@@ -30,4 +29,7 @@
       <axis xyz="0 1 0" />
     </joint>
+    <!-- TODO:
+         - Gazebo: controller for wheel differential drive
+    -->
   </xacro:macro>
 </robot>

Commit message: Fix typos & missing tags for caster in base

File: mark_description/urdf/base.urdf.xacro (robot description, xacro)
@@ -13,7 +13,9 @@
   <xacro:property name="caster_origin" value="-0.073 0 -0.02" />
   <xacro:property name="caster_geom">
-    <sphere radius="0.010" />
+    <geometry>
+      <sphere radius="0.010" />
+    </geometry>
   </xacro:property>
-  <xacro:property name="base_inertia">
+  <xacro:property name="caster_inertial">
     <inertial>
       <mass value="0.5" />

Commit message: Model ultrasonic sensor (optional with arg)

File: mark_description/urdf/base.urdf.xacro (robot description, xacro)
@@ -17,5 +17,5 @@
     </geometry>
   </xacro:property>
-  <xacro:property name="caster_inertial">
+  <xacro:property name="caster_inertia">
     <inertial>
       <mass value="0.5" />
@@ -52,5 +52,5 @@
         <xacro:insert_block name="caster_geom" />
       </collision>
-      <xacro:insert_block name="caster_inertial" />
+      <xacro:insert_block name="caster_inertia" />
     </link>
     <joint name="caster_to_base_joint" type="fixed">

File: mark_description/urdf/mark.urdf.xacro (robot description, xacro)
@@ -1,4 +1,6 @@
 <?xml version='1.0'?>
 <robot name="mark" xmlns:xacro="http://ros.org/wiki/xacro">
+  <!-- Parameters -->
+  <xacro:arg name="ultrasonic_sensor_enabled" default="true" />
   <!-- Includes -->
   <xacro:include filename="$(find mark_description)/urdf/inertial.urdf.xacro" />
@@ -7,4 +9,5 @@
   <xacro:include filename="$(find mark_description)/urdf/wheel.urdf.xacro" />
   <xacro:include filename="$(find mark_description)/urdf/camera.urdf.xacro" />
+  <xacro:include filename="$(find mark_description)/urdf/ultrasonic.urdf.xacro" />
   <!-- Base/chassis -->
   <xacro:mark_base></xacro:mark_base>
@@ -20,6 +23,11 @@
     <origin xyz="0.06 0.0 0.023" rpy="0 0 0" />
   </xacro:mark_camera>
+  <!-- Ultrasonic sensor (if requied) -->
+  <xacro:if value="$(arg ultrasonic_sensor_enabled)">
+    <xacro:mark_ultrasonic_sensor>
+      <origin xyz="0.083 0.0 -0.006" rpy="0 0 0" />
+    </xacro:mark_ultrasonic_sensor>
+  </xacro:if>
   <!-- TODO:
-       - Ultrasonic sensor (controlled by arg)
        - Gripper (controller by arg)
   -->
