Commit message: Modify URDF description to work with Unity
The robot model finally works with a simulator!

File: mark_description/urdf/base.urdf.xacro (robot description, xacro)
@@ -4,10 +4,4 @@
       <box size="0.166 0.125 0.036" />
     </geometry>
-  </xacro:property>
-  <xacro:property name="base_inertia">
-    <inertial>
-      <mass value="0.62" />
-      <xacro:box_inertia m="0.62" d="0.166" w="0.125" h="0.036" />
-    </inertial>
   </xacro:property>
   <xacro:property name="caster_origin" value="-0.073 0 -0.02" />
@@ -17,11 +11,6 @@
     </geometry>
   </xacro:property>
-  <xacro:property name="caster_inertia">
-    <inertial>
-      <mass value="0.5" />
-      <xacro:sphere_inertia m="0.5" r="0.010" />
-    </inertial>
-  </xacro:property>
   <xacro:macro name="mark_base">
+    <link name="world" />
     <!-- Base -->
     <link name="base_link">
@@ -34,12 +23,10 @@
       </collision>
     </link>
-    <!-- Inertial link stores the robot's inertial information
-         Has to be defined separately because root links can't have intertial information directly -->
-    <link name="inertial_link">
-      <xacro:insert_block name="base_inertia" />
-    </link>
-    <joint name="inertial_joint" type="fixed">
-      <parent link="base_link" />
-      <child link="inertial_link" />
+    <!-- Join the base to the "world" which will act as the unifying link of the whole robot
+         This is needed for the robot to be imported properly in Unity -->
+    <joint name="joint_world" type="fixed">
+        <parent link="world" />
+        <child link="base_link" />
+        <origin xyz="0 0 0" rpy="0 0 0" />
     </joint>
     <!-- Caster (i.e. back support) -->
@@ -52,5 +39,4 @@
         <xacro:insert_block name="caster_geom" />
       </collision>
-      <xacro:insert_block name="caster_inertia" />
     </link>
     <joint name="caster_to_base_joint" type="fixed">

File: mark_description/urdf/camera.urdf.xacro (robot description, xacro)
@@ -4,10 +4,4 @@
       <cylinder length="0.01" radius="0.0225" />
     </geometry>
-  </xacro:property>
-  <xacro:property name="camera_pan_support_inertia">
-    <inertial>
-      <mass value="0.005" />
-      <xacro:cylinder_inertia m="0.005" r="0.0225" h="0.01" />
-    </inertial>
   </xacro:property>
   <xacro:property name="camera_tilt_support_geom">
@@ -18,10 +12,4 @@
   <xacro:property name="camera_tilt_support_joint_pose">
     <origin xyz="0.005 0 0.015" rpy="0 0 0" />
-  </xacro:property>
-  <xacro:property name="camera_tilt_support_inertia">
-    <inertial>
-      <mass value="0.005" />
-      <xacro:box_inertia m="0.005" d="0.035" w="0.025" h="0.02" />
-    </inertial>
   </xacro:property>
   <xacro:property name="camera_lateral_support_geom">
@@ -34,5 +22,5 @@
   </xacro:property>
   <xacro:property name="camera_left_lateral_support_link_pose">
-    <origin xyz="0 0 0.021" rpy="0 0 0" />
+    <origin xyz="-0.009 0 -0.0155" rpy="0 0 0" />
   </xacro:property>
   <xacro:property name="camera_right_lateral_support_joint_pose">
@@ -41,10 +29,4 @@
   <xacro:property name="camera_left_lateral_support_joint_pose">
     <origin xyz="0.009 -0.013 0" rpy="0 0 0" />
-  </xacro:property>
-  <xacro:property name="camera_lateral_support_inertia">
-    <inertial>
-      <mass value="0.005" />
-      <xacro:box_inertia m="0.005" d="0.012" w="0.001" h="0.057" />
-    </inertial>
   </xacro:property>
   <xacro:property name="camera_lens_support_geom">
@@ -55,10 +37,4 @@
   <xacro:property name="camera_lens_support_joint_pose">
     <origin xyz="0 -0.013 0.0365" rpy="0 0 0" />
-  </xacro:property>
-  <xacro:property name="camera_lens_support_inertia">
-    <inertial>
-      <mass value="0.005" />
-      <xacro:box_inertia m="0.005" d="0.012" w="0.025" h="0.026" />
-    </inertial>
   </xacro:property>
   <xacro:property name="camera_lens_geom">
@@ -71,37 +47,4 @@
     <origin xyz="0.012 0 0.003" rpy="0 1.560795 0" />
   </xacro:property>
-  <xacro:property name="camera_lens_inertia">
-    <inertial>
-      <mass value="0.0025" />
-      <xacro:cylinder_inertia m="0.0025" r="0.006" h="0.012"  />
-    </inertial>
-  </xacro:property>
-  <!-- Macro for lateral support for holding the lens support -->
-  <xacro:macro name="camera_lateral_support" params="prefix mimic_joint:='none' *link_pose *joint_pose">
-    <link name="camera_${prefix}_lateral_support_link">
-      <visual>
-        <xacro:insert_block name="link_pose" />
-        <xacro:insert_block name="camera_lateral_support_geom" />
-        <material name="black" />
-      </visual>
-      <collision>
-        <xacro:insert_block name="link_pose" />
-        <xacro:insert_block name="camera_lateral_support_geom" />
-      </collision>
-      <xacro:insert_block name="camera_lateral_support_inertia" />
-    </link>
-    <joint name="camera_${prefix}_lateral_support_to_tilt_support_joint" type="revolute">
-      <parent link="camera_tilt_support_link" />
-      <child link="camera_${prefix}_lateral_support_link" />
-      <xacro:insert_block name="joint_pose" />
-      <!-- Rotation on the y-axis (tilt) -->
-      <axis xyz="0 1 0" />
-      <!-- -75 to 90 degrees -->
-      <limit lower="-1.309" upper="1.560795" effort="1.0" velocity="1.0" />
-      <xacro:if value="${mimic_joint != 'none'}" >
-        <mimic joint="${mimic_joint}" />
-      </xacro:if>
-    </joint>
-  </xacro:macro>
   <!-- Full camera macro -->
   <xacro:macro name="mark_camera" params="*main_camera_joint_pose">
@@ -115,5 +58,4 @@
         <xacro:insert_block name="camera_pan_support_geom" />
       </collision>
-      <xacro:insert_block name="camera_pan_support_inertia" />
     </link>
     <joint name="camera_pan_support_to_base_joint" type="revolute">
@@ -135,5 +77,4 @@
         <xacro:insert_block name="camera_tilt_support_geom" />
       </collision>
-      <xacro:insert_block name="camera_tilt_support_inertia" />
     </link>
     <joint name="camera_tilt_support_to_pan_support_joint" type="fixed">
@@ -142,13 +83,25 @@
       <xacro:insert_block name="camera_tilt_support_joint_pose" />
     </joint>
-    <!-- Lateral supports for lens that provide tilting -->
-    <xacro:camera_lateral_support prefix="right">
-      <xacro:insert_block name="camera_right_lateral_support_link_pose" />
+    <!-- Lateral support for lens that provide tilting (only the right will move) -->
+    <link name="camera_right_lateral_support_link">
+      <visual>
+        <xacro:insert_block name="camera_right_lateral_support_link_pose" />
+        <xacro:insert_block name="camera_lateral_support_geom" />
+        <material name="black" />
+      </visual>
+      <collision>
+        <xacro:insert_block name="camera_right_lateral_support_link_pose" />
+        <xacro:insert_block name="camera_lateral_support_geom" />
+      </collision>
+    </link>
+    <joint name="camera_right_lateral_support_to_tilt_support_joint" type="revolute">
+      <parent link="camera_tilt_support_link" />
+      <child link="camera_right_lateral_support_link" />
       <xacro:insert_block name="camera_right_lateral_support_joint_pose" />
-    </xacro:camera_lateral_support>
-    <xacro:camera_lateral_support prefix="left" mimic_joint="camera_right_lateral_support_to_tilt_support_joint">
-      <xacro:insert_block name="camera_left_lateral_support_link_pose" />
-      <xacro:insert_block name="camera_left_lateral_support_joint_pose" />
-    </xacro:camera_lateral_support>
+      <!-- Rotation on the y-axis (tilt) -->
+      <axis xyz="0 1 0" />
+      <!-- -75 to 90 degrees -->
+      <limit lower="-1.309" upper="1.560795" effort="1.0" velocity="1.0" />
+    </joint>
     <!-- Lens support -->
     <link name="camera_lens_support_link">
@@ -160,5 +113,4 @@
         <xacro:insert_block name="camera_lens_support_geom" />
       </collision>
-      <xacro:insert_block name="camera_lens_support_inertia" />
     </link>
     <joint name="camera_lens_support_to_lateral_support_joint" type="fixed">
@@ -166,4 +118,25 @@
       <child link="camera_lens_support_link" />
       <xacro:insert_block name="camera_lens_support_joint_pose" />
+    </joint>
+    <!-- Left lateral support for lens that does not move on its own
+         Movement is controlled by thr right lateral support
+         We add this so that it matches the visual design of the robot -->
+    <link name="camera_left_lateral_support_link">
+      <visual>
+        <xacro:insert_block name="camera_left_lateral_support_link_pose" />
+        <xacro:insert_block name="camera_lateral_support_geom" />
+        <material name="black" />
+      </visual>
+      <collision>
+        <xacro:insert_block name="camera_left_lateral_support_link_pose" />
+        <xacro:insert_block name="camera_lateral_support_geom" />
+      </collision>
+    </link>
+    <!-- Join the lateral support with a fixed joint so that it moves with the whole
+         camera lens when the right support moves -->
+    <joint name="camera_left_lateral_support_to_lens_support_joint" type="fixed">
+      <parent link="camera_lens_support_link" />
+      <child link="camera_left_lateral_support_link" />
+      <xacro:insert_block name="camera_left_lateral_support_joint_pose" />
     </joint>
     <!-- Camera lens -->
@@ -176,5 +149,4 @@
         <xacro:insert_block name="camera_lens_geom" />
       </collision>
-      <xacro:insert_block name="camera_lens_inertia" />
     </link>
     <joint name="camera_lens_to_lens_support_joint" type="fixed">
@@ -183,9 +155,4 @@
       <xacro:insert_block name="camera_lens_joint_pose" />
     </joint>
-    <!-- TODO:
-         - Gazebo:
-           - Camera sensor
-           - Controller for pan and tilt servos
-    -->
   </xacro:macro>
 </robot>

File: mark_description/urdf/gripper.urdf.xacro (robot description, xacro)
@@ -7,12 +7,7 @@
   <xacro:property name="gripper_base_collision">
     <geometry>
-      <box size="0.015 0.073 0.035" />
+      <box size="0.015 0.073 0.03" />
     </geometry>
-  </xacro:property>
-  <xacro:property name="gripper_base_inertia">
-    <inertial>
-      <mass value="0.001" />
-      <xacro:box_inertia m="0.001" d="0.015" w="0.073" h="0.035" />
-    </inertial>
+    <origin xyz="0.0613 0 0.016" rpy="0 0 0" />
   </xacro:property>
   <xacro:property name="gripper_arm_collision">
@@ -23,4 +18,7 @@
   <xacro:property name="gripper_arm_a_link_pose">
     <origin xyz="0.015 0 0" rpy="0 0 0" />
+  </xacro:property>
+  <xacro:property name="gripper_arm_a_collision_pose">
+    <origin xyz="0.031 0 0" rpy="0 0 0" />
   </xacro:property>
   <xacro:property name="gripper_arm_b_link_pose">
@@ -33,12 +31,6 @@
     <origin xyz="0.06 0.01 0" rpy="0 0 0" />
   </xacro:property>
-  <xacro:property name="gripper_arm_inertia">
-    <inertial>
-      <mass value="0.001" />
-      <xacro:box_inertia m="0.001" d="0.07" w="0.01" h="0.01" />
-    </inertial>
-  </xacro:property>
   <!-- Macro for gripper arms -->
-  <xacro:macro name="gripper_arm" params="prefix mimic_joint:='none' *link_pose *joint_pose">
+  <xacro:macro name="gripper_arm" params="prefix anchor_rotation *link_pose *collision_pose *joint_pose">
     <link name="gripper_arm_${prefix}_link">
       <visual>
@@ -49,8 +41,7 @@
       </visual>
       <collision>
-        <xacro:insert_block name="link_pose" />
+        <xacro:insert_block name="collision_pose" />
         <xacro:insert_block name="gripper_arm_collision" />
       </collision>
-      <xacro:insert_block name="gripper_arm_inertia" />
     </link>
     <joint name="gripper_arm_${prefix}_to_gripper_base_joint" type="revolute">
@@ -59,13 +50,7 @@
       <xacro:insert_block name="joint_pose" />
       <!-- Rotation on the z-axis -->
-      <axis xyz="0 0 1" />
+      <axis xyz="0 0 ${anchor_rotation}" />
       <!-- -90 to ~5 degrees (radians) so that the two arms can meet -->
       <limit lower="-1.560795" upper="0.09" effort="1.0" velocity="1.0" />
-      <xacro:if value="${mimic_joint != 'none'}" >
-        <!-- We use a multiplier of -1 to make the joints move opposite of each other
-             This allows both arms to open and close correctly
-        -->
-        <mimic joint="${mimic_joint}" multiplier="-1.0"/>
-      </xacro:if>
     </joint>
   </xacro:macro>
@@ -79,5 +64,4 @@
         <xacro:insert_block name="gripper_base_collision" />
       </collision>
-      <xacro:insert_block name="gripper_base_inertia" />
     </link>
     <joint name="gripper_base_to_robot_base_link" type="fixed">
@@ -86,16 +70,28 @@
       <xacro:insert_block name="gripper_base_joint_pose" />
     </joint>
-    <!-- Two gripper arms -->
-    <xacro:gripper_arm prefix="a">
+    <!-- Two gripper arms
+         We need a separate pose for the collision because if we use the link pose,
+         the collision mesh ends up not aligning properly; not sure why though.
+         For the gripper b side we can use the same pose as the link because
+         it seems the 3D model matches it perfectly -->
+    <xacro:gripper_arm prefix="a" anchor_rotation="1">
       <xacro:insert_block name="gripper_arm_a_link_pose" />
+      <xacro:insert_block name="gripper_arm_a_collision_pose" />
       <xacro:insert_block name="gripper_arm_a_joint_pose" />
     </xacro:gripper_arm>
-    <xacro:gripper_arm prefix="b" mimic_joint="gripper_arm_a_to_gripper_base_joint">
+    <xacro:gripper_arm prefix="b" anchor_rotation="-1">
+      <xacro:insert_block name="gripper_arm_b_link_pose" />
       <xacro:insert_block name="gripper_arm_b_link_pose" />
       <xacro:insert_block name="gripper_arm_b_joint_pose" />
     </xacro:gripper_arm>
-    <!-- TODO:
-         - Gazebo: controller for gripper arm servo
-    -->
+    <!--Disable collisions between the grippers, the base and the ultrasonic sensor
+        This allows the grippers to open and close smoothly
+        See: https://github.com/Unity-Technologies/Unity-Robotics-Hub/blob/main/tutorials/urdf_importer/urdf_appendix.md#disable-collision-support -->
+    <disable_collision link1="gripper_arm_a_link" link2="gripper_base_link"></disable_collision>
+    <disable_collision link1="gripper_arm_b_link" link2="gripper_base_link"></disable_collision>
+    <disable_collision link1="gripper_arm_a_link" link2="ultrasonic_sensor_base_link"></disable_collision>
+    <disable_collision link1="gripper_arm_b_link" link2="ultrasonic_sensor_base_link"></disable_collision>
+    <disable_collision link1="gripper_arm_a_link" link2="ultrasonic_sensor_left_link"></disable_collision>
+    <disable_collision link1="gripper_arm_b_link" link2="ultrasonic_sensor_right_link"></disable_collision>
   </xacro:macro>
 </robot>

File: mark_description/urdf/ultrasonic.urdf.xacro (robot description, xacro)
@@ -4,10 +4,4 @@
       <box size="0.001 0.047 0.03" />
     </geometry>
-  </xacro:property>
-  <xacro:property name="ultrasonic_sensor_base_inertia">
-    <inertial>
-      <mass value="0.005" />
-      <xacro:box_inertia m="0.005" d="0.001" w="0.045" h="0.023" />
-    </inertial>
   </xacro:property>
   <xacro:property name="ultrasonic_sensor_geom">
@@ -24,10 +18,4 @@
     <origin xyz="0.0076 -0.012 -0.005" rpy="0 1.560795 0" />
   </xacro:property>
-  <xacro:property name="ultrasonic_sensor_inertia">
-    <inertial>
-      <mass value="0.005" />
-      <xacro:cylinder_inertia m="0.005" r="0.0075" h="0.013" />
-    </inertial>
-  </xacro:property>
   <!-- Macro for lateral support for holding the lens support -->
   <xacro:macro name="ultrasonic_sensor" params="prefix *joint_pose">
@@ -40,5 +28,4 @@
         <xacro:insert_block name="ultrasonic_sensor_geom" />
       </collision>
-      <xacro:insert_block name="ultrasonic_sensor_inertia" />
     </link>
     <joint name="ultrasonic_sensor_${prefix}_to_sensor_base_joint" type="fixed">
@@ -58,5 +45,4 @@
         <xacro:insert_block name="ultrasonic_sensor_base_geom" />
       </collision>
-      <xacro:insert_block name="ultrasonic_sensor_base_inertia" />
     </link>
     <joint name="ultrasonic_sensor_base_to_parent_link" type="fixed">
@@ -72,7 +58,4 @@
       <xacro:insert_block name="ultrasonic_sensor_left_joint_pose" />
     </xacro:ultrasonic_sensor>
-    <!-- TODO:
-         - Gazebo: ultrasonic sensors
-    -->
   </xacro:macro>
 </robot>

File: mark_description/urdf/wheel.urdf.xacro (robot description, xacro)
@@ -14,11 +14,7 @@
         <origin xyz="0 0 0" rpy="1.560795 0 0" />
         <geometry>
-          <cylinder length="0.062" radius="0.031" />
+          <cylinder length="0.027" radius="0.031" />
         </geometry>
       </collision>
-      <inertial>
-        <mass value="0.5" />
-        <xacro:cylinder_inertia m="0.5" r="0.031" h="0.062" />
-      </inertial>
     </link>
     <joint name="joint_${wheel_prefix}_wheel" type="continuous">
@@ -29,7 +25,4 @@
       <axis xyz="0 1 0" />
     </joint>
-    <!-- TODO:
-         - Gazebo: controller for wheel differential drive
-    -->
   </xacro:macro>
 </robot>

Commit message: Update position of caster to touch ground in URDF
The caster has to touch the ground to stabilize the robot
and keep it straight. Otherwise, it would cause the robot
to tilt upwards.

File: mark_description/urdf/base.urdf.xacro (robot description, xacro)
@@ -5,5 +5,5 @@
     </geometry>
   </xacro:property>
-  <xacro:property name="caster_origin" value="-0.073 0 -0.02" />
+  <xacro:property name="caster_origin" value="-0.073 0 -0.025" />
   <xacro:property name="caster_geom">
     <geometry>
